Commit message: Add files via upload

File: urdf/rpi_robot.urdf.xacro (robot description, xacro)
@@ -275,5 +275,5 @@
       <parent link="base_link"/>
       <child link="laser_frame"/>
-      <origin xyz="0.3 0 0.15" rpy="0 0 0"/>
+      <origin xyz="0.3 0 0.1" rpy="0 0 0"/>
   </joint>
   <link name="laser_frame">
@@ -300,5 +300,5 @@
       <sensor name="laser" type="ray">
           <pose> 0 0 0 0 0 0 </pose>
-          <visualize>true</visualize>
+          <visualize>false</visualize>
           <update_rate>30</update_rate>
           <ray>
@@ -324,3 +324,46 @@
       </sensor>
   </gazebo>
+  <!-- Camera -->
+   <joint name="camera_joint" type="fixed">
+        <parent link="base_link"/>
+        <child link="camera_link"/>
+        <origin xyz="0.4 0 0" rpy="0 0 0"/>
+    </joint>
+    <link name="camera_link">
+        <visual>
+            <geometry>
+                <box size="0.010 0.03 0.03"/>
+            </geometry>
+            <material name="red"/>
+        </visual>
+    </link>
+    <joint name="camera_optical_joint" type="fixed">
+        <parent link="camera_link"/>
+        <child link="camera_link_optical"/>
+        <origin xyz="0 0 0" rpy="${-pi/2} 0 ${-pi/2}"/>
+    </joint>
+    <link name="camera_link_optical"></link>
+    <gazebo reference="camera_link">
+        <material>Gazebo/Red</material>
+        <sensor name="camera" type="camera">
+            <pose> 0 0 0 0 0 0 </pose>
+            <visualize>true</visualize>
+            <update_rate>10</update_rate>
+            <camera>
+                <horizontal_fov>1.089</horizontal_fov>
+                <image>
+                    <format>R8G8B8</format>
+                    <width>640</width>
+                    <height>480</height>
+                </image>
+                <clip>
+                    <near>0.05</near>
+                    <far>8.0</far>
+                </clip>
+            </camera>
+            <plugin name="camera_controller" filename="libgazebo_ros_camera.so">
+                <frame_name>camera_link_optical</frame_name>
+            </plugin>
+        </sensor>
+    </gazebo>
 </robot>
